File: PCB/Solver_Shield/MCXA153_Solver_Shield.kicad_pcb (KiCad board)
At the start: 2 copper layers, 91.4 x 54.6 mm, 22 parts, among them IC1 74ALVC00D-Q100J, IC2 74ALVC00D-Q100J, IC3 74ALVC00D-Q100J, IC4 ULN2003ANSRE4, IC5 ISO6721RBDR, IC6 74ALVC00D-Q100J, J1 SSQ-108-03-T-D, J2 SSQ-110-03-T-D, J3 SSQ-108-03-T-D, J4 SSQ-106-03-T-D

Commit message: update PCB
Connections:
- IC3 pad 11: unconnected-(IC3-4Y-Pad11) -> /EN_ALL
- IC3 pad 12: unconnected-(IC3-4A-Pad12) -> /P2-7/TRIG10
- IC3 pad 13: unconnected-(IC3-4B-Pad13) -> /P2-7/TRIG10
- U4 pad 7: GND -> /EN_ALL
Routing:
- net /EN_ALL: track 0.00 -> 39.3 mm
- net /P2-7/TRIG10: track 0.00 -> 29.0 mm
- net VDD_5V: track 189.2 -> 178.2 mm, vias 6 -> 5
- net /P3-14/PWM0-X2: track 47.3 -> 47.9 mm
- net GND: vias 10 -> 12
