File: PCB/Solver_Shield/MCXA153_Solver_Shield.kicad_sch (KiCad schematic)
At the start: 22 parts, among them IC1 74ALVC00D-Q100J, IC2 74ALVC00D-Q100J, IC3 74ALVC00D-Q100J, IC4 ULN2003ANSRE4, IC5 ISO6721RBDR, IC6 74ALVC00D-Q100J, J1 ${ALTIUM_VALUE}, J2 ${ALTIUM_VALUE}, J3 ${ALTIUM_VALUE}, J4 ${ALTIUM_VALUE}

Commit message: update PCB
Parts:
- R2: value R -> 10k
Connections:
- net GND: no longer U4.7 (EN_ALL)
- net P2-7/TRIG10: now also IC3.12 (4A), IC3.13 (4B)
- net EN_ALL: now reaches IC3.11 (4Y)
- net EN_ALL: now also U4.7 (EN_ALL)
Other:
- note added: "MCXA153"
- company: (none) -> Hochschule Wismar
- title: (none) -> Projektseminar Speed_Solver
- moved on the sheet: D1, IC1, IC4, IC5, IC6, J1, J2, J3, J4, R2, U1, U10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
